File: Circuit Boards/XBEEadded/CntrlBoard.brd (EAGLE design)
At the start: 101.6 x 81.3 mm, 49 parts, among them P1 22-23-2021, P10 3PIN2MMPITCH, P11 3PIN2MMPITCH, P12 DF3A-2P-2DSA, P13 DF3A-2P-2DSA, P14 DF3A-2P-2DSA, P15 DF3A-2P-2DSA, P16 DF3A-2P-2DSA, P17 DF3A-2P-2DSA, P18 DF3A-2P-2DSA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

Commit message: Added updates 3, 4, 6, and 9 from UpdatesToDo.txt
Parts:
- moved LED3 94.6 mm to (98.4, 18.4), turned to 0 degrees
- moved R7 5.71 mm to (51.4, 34.3)
- moved VR1 4.45 mm to (52.7, 39.4)
- moved U$2 3.81 mm to (47.0, 35.6)
Routing:
- net N$12: track 7.01 -> 171.8 mm
- net VCC: track 175.4 -> 190.5 mm, vias 5 -> 4
- net +5V: track 201.4 -> 191.9 mm
- net STDBY_N: track 39.4 -> 43.2 mm
- net PWMB: track 39.4 -> 35.6 mm
- net PWMA: track 21.6 -> 17.8 mm
- net BIN2: track 39.4 -> 43.2 mm
- net BIN1: track 39.4 -> 43.2 mm
- net AIN2: track 39.4 -> 43.2 mm
- net AIN1: track 39.4 -> 43.2 mm
- net N$20: track 43.9 -> 46.4 mm, vias 1 -> 2
- net N$18: track 41.7 -> 44.3 mm, vias 1 -> 2
- net N$17: track 49.4 -> 51.9 mm, vias 1 -> 2
- net N$19: track 43.4 -> 45.9 mm, vias 1 -> 2
- net N$21: track 8.74 -> 7.17 mm
Other:
- board text added: "24V"
- board text added: "24V IN"
- board text added: "24V OUT"
- board text added: "24V OUTS"
- board text added: "5V"
- board text added: "5V ENABLE"
- board text added: "5V OUT"
- board text added: "5V OUTS"
- board text added: "IMU SERIAL"
- board text added: "LINEAR"
- board text added: "PUMP DIR."
- board text added: "PUMP DIRECTION"
- board text added: "PUMP ON"
- board text added: "ROTARY"
