File: Circuit Boards/UpdatedMainBoard/CntrlBoard.brd (EAGLE design)
At the start: 101.6 x 81.3 mm, 63 parts, among them P1 22-23-2021, P10 3MM2MMLOCKING, P11 3MM2MMLOCKING, P12 DF3A-2P-2DSA, P13 DF3A-2P-2DSA, P14 DF3A-2P-2DSA, P15 DF3A-2P-2DSA, P16 DF3A-2P-2DSA, P17 DF3A-2P-2DSA, P18 DF3A-2P-2DSA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

Commit message: Updated main board again
Parts:
- added LED5: GRN, led:CHIPLED_1206
- added LED6: RED, led:CHIPLED_1206
- added R15: 5K0, resistor:R1206
- added R16, R17, R18: 1K0, resistor:R1206
Connections:
- new net N$23: LED6.C, U1.42
- new net N$28: LED5.A, R17.2
- new net N$29: LED6.A, R18.2
- new net N$3: LED5.C, U1.40
- new net VIN_READBACK: R15.2, R16.1, U1.A13
- net +5V: now also R17.1, R18.1
- net GND: now also R16.2
- net VCC: now also R15.1
Routing:
- net +5V: track 250.3 -> 321.0 mm
- net VIN_READBACK: track 0.00 -> 10.0 mm, vias 0 -> 1
- net VCC: track 265.4 -> 271.9 mm
- net GND: track 585.7 -> 591.5 mm, vias 8 -> 9
- net N$3: track 0.00 -> 3.33 mm
- net N$23: track 0.00 -> 3.33 mm
- net N$29: track 0.00 -> 3.18 mm
- net N$28: track 0.00 -> 3.18 mm
Other:
- board text added: "HLTHY"
Changed lines of the file:
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@@
 <text x="64.77" y="55.245" size="1.27" layer="1" font="vector">PUMP
 DIRECTION</text>
-<text x="86.995" y="45.72" size="1.27" layer="1" font="vector" rot="R90">LINEAR</text>
-<text x="86.995" y="37.465" size="1.27" layer="1" font="vector" rot="R90">ROTARY</text>
+<text x="78.74" y="46.99" size="1.27" layer="1" font="vector" rot="R90">LINEAR</text>
+<text x="78.74" y="35.56" size="1.27" layer="1" font="vector" rot="R90">ROTARY</text>
 <text x="1.27" y="77.47" size="1.27" layer="1" font="vector">5V OUT</text>
 <text x="13.335" y="8.255" size="1.27" layer="1" font="vector">24V IN</text>
@@
 <text x="15.24" y="70.485" size="1.27" layer="1" font="vector" rot="R90">5V ENABLE</text>
 <text x="19.685" y="16.51" size="1.27" layer="1" font="vector">ROUGHIE 2 MAIN BOARD V2</text>
+<text x="91.44" y="46.355" size="1.27" layer="1" font="vector" rot="R90">HLTHY</text>
 </plain>
 <attributes>
@@
 <element name="C9" library="resistor" package="C1210K" value="0U1" x="59.055" y="31.75" rot="MR90"/>
 <element name="P22" library="con-3m" package="6PIN2ROWARDUINO" value="6PIN2ROWARDUINO" x="20.955" y="22.86"/>
+<element name="R15" library="resistor" package="R1206" value="5K0" x="81.915" y="28.575" rot="R270"/>
+<element name="R16" library="resistor" package="R1206" value="1K0" x="85.09" y="28.575" rot="R90"/>
+<element name="LED5" library="led" package="CHIPLED_1206" value="GRN" x="88.9" y="44.45" rot="R270"/>
+<element name="LED6" library="led" package="CHIPLED_1206" value="RED" x="88.9" y="41.91" rot="R270"/>
+<element name="R17" library="resistor" package="R1206" value="1K0" x="86.995" y="48.895" rot="R270"/>
+<element name="R18" library="resistor" package="R1206" value="1K0" x="86.995" y="37.465" rot="R90"/>
 </elements>
 <signals>
@@
 <wire x1="83.185" y1="36.83" x2="83.185" y2="33.02" width="1.016" layer="16"/>
 <wire x1="83.185" y1="33.02" x2="83.185" y2="26.67" width="1.016" layer="16"/>
-<wire x1="83.185" y1="26.67" x2="93.98" y2="26.67" width="1.016" layer="16"/>
+<wire x1="83.185" y1="26.67" x2="87.63" y2="26.67" width="1.016" layer="16"/>
+<wire x1="87.63" y1="26.67" x2="93.98" y2="26.67" width="1.016" layer="16"/>
 <wire x1="48.26" y1="54.61" x2="50.8" y2="54.61" width="1.016" layer="16"/>
 <wire x1="50.8" y1="54.61" x2="50.8" y2="52.705" width="1.016" layer="16"/>
@@
 <wire x1="26.035" y1="25.4" x2="34.29" y2="25.4" width="1.016" layer="16"/>
 <wire x1="34.29" y1="25.4" x2="34.29" y2="30.48" width="1.016" layer="16"/>
+<contactref element="R16" pad="2"/>
+<wire x1="85.09" y1="29.997" x2="87.63" y2="29.997" width="0.254" layer="1"/>
+<wire x1="87.63" y1="29.997" x2="87.63" y2="29.845" width="0.254" layer="1"/>
+<via x="87.63" y="29.845" extent="1-16" drill="0.7" shape="square"/>
+<wire x1="87.63" y1="29.845" x2="87.63" y2="26.67" width="0.254" layer="16"/>
 </signal>
 <signal name="N$1">
@@
 <wire x1="16.51" y1="20.55" x2="16.51" y2="22.86" width="0.254" layer="16"/>
 <wire x1="20.955" y1="22.86" x2="16.51" y2="22.86" width="1.016" layer="16"/>
+<contactref element="R15" pad="1"/>
+<wire x1="81.915" y1="29.997" x2="78.105" y2="29.997" width="0.254" layer="1"/>
+<wire x1="78.105" y1="29.997" x2="78.105" y2="27.305" width="0.254" layer="1"/>
 </signal>
 <signal name="N$4">
@@
 <wire x1="21.59" y1="38.735" x2="21.995" y2="38.735" width="1.016" layer="16"/>
 <wire x1="21.995" y1="38.735" x2="21.995" y2="42.545" width="1.016" layer="16"/>
+<contactref element="R17" pad="1"/>
+<contactref element="R18" pad="1"/>
+<wire x1="86.995" y1="50.317" x2="86.995" y2="54.61" width="0.254" layer="1"/>
+<wire x1="86.995" y1="54.61" x2="80.645" y2="54.61" width="0.254" layer="1"/>
+<wire x1="80.645" y1="54.61" x2="63.5" y2="54.61" width="0.254" layer="1"/>
+<wire x1="63.5" y1="54.61" x2="63.5" y2="55.88" width="0.254" layer="1"/>
+<wire x1="63.5" y1="55.88" x2="50.165" y2="55.88" width="0.254" layer="1"/>
+<wire x1="50.165" y1="55.88" x2="50.165" y2="58.42" width="0.254" layer="1"/>
+<wire x1="50.165" y1="58.42" x2="49.3" y2="58.42" width="0.254" layer="1"/>
+<wire x1="86.995" y1="36.043" x2="80.645" y2="36.043" width="0.254" layer="1"/>
+<wire x1="80.645" y1="36.043" x2="80.645" y2="54.61" width="0.254" layer="1"/>
 </signal>
 <signal name="N$12">
@@
 <contactref element="LED3" pad="C"/>
 <wire x1="98.425" y1="20.165" x2="98.425" y2="24.13" width="0.254" layer="1"/>
-<wire x1="98.425" y1="24.13" x2="83.185" y2="24.13" width="0.254" layer="1"/>
-<wire x1="83.185" y1="24.13" x2="83.185" y2="32.385" width="0.254" layer="1"/>
-<wire x1="83.185" y1="32.385" x2="50.8" y2="32.385" width="0.254" layer="1"/>
+<wire x1="98.425" y1="24.13" x2="89.535" y2="24.13" width="0.254" layer="1"/>
+<wire x1="89.535" y1="24.13" x2="89.535" y2="32.385" width="0.254" layer="1"/>
+<wire x1="89.535" y1="32.385" x2="50.8" y2="32.385" width="0.254" layer="1"/>
 <wire x1="50.8" y1="32.385" x2="50.8" y2="38.1" width="0.254" layer="1"/>
 <wire x1="50.8" y1="38.1" x2="46.355" y2="38.1" width="0.254" layer="1"/>
@@
 <wire x1="85.09" y1="7.62" x2="82.55" y2="7.62" width="1.016" layer="16"/>
 </signal>
+<signal name="VIN_READBACK">
+<contactref element="R15" pad="2"/>
+<contactref element="R16" pad="1"/>
+<contactref element="U1" pad="A13"/>
+<wire x1="81.915" y1="27.153" x2="85.09" y2="27.153" width="0.4064" layer="1"/>
+<wire x1="86.36" y1="21.59" x2="86.36" y2="24.13" width="0.254" layer="16"/>
+<via x="86.36" y="24.13" extent="1-16" drill="0.7" shape="square"/>
+<wire x1="86.36" y1="24.13" x2="85.09" y2="24.13" width="0.254" layer="1"/>
+<wire x1="85.09" y1="24.13" x2="85.09" y2="27.153" width="0.254" layer="1"/>
+</signal>
+<signal name="N$3">
+<contactref element="LED5" pad="C"/>
+<contactref element="U1" pad="40"/>
+<wire x1="93.98" y1="44.45" x2="90.65" y2="44.45" width="0.254" layer="1"/>
+</signal>
+<signal name="N$23">
+<contactref element="U1" pad="42"/>
+<contactref element="LED6" pad="C"/>
+<wire x1="93.98" y1="41.91" x2="90.65" y2="41.91" width="0.254" layer="1"/>
+</signal>
+<signal name="N$28">
+<contactref element="LED5" pad="A"/>
+<contactref element="R17" pad="2"/>
+<wire x1="86.995" y1="47.473" x2="87.15" y2="47.473" width="0.254" layer="1"/>
+<wire x1="87.15" y1="47.473" x2="87.15" y2="44.45" width="0.254" layer="1"/>
+</signal>
+<signal name="N$29">
+<contactref element="LED6" pad="A"/>
+<contactref element="R18" pad="2"/>
+<wire x1="87.15" y1="41.91" x2="86.995" y2="41.91" width="0.254" layer="1"/>
+<wire x1="86.995" y1="41.91" x2="86.995" y2="38.887" width="0.254" layer="1"/>
+</signal>
 </signals>
