File: Circuit Boards/Xbee_SD_etc_Shield/additionalShield.brd (EAGLE design)
At the start: 85.1 x 53.3 mm, 52 parts, among them P1 DF3A-2P-2DSA, P2 DF3A-2P-2DSA, Q1 BSS123, Q2 BSS123, Q3 BSS123, U2 XBEE-1B3, U3 V_REG_LDOSMD, U4 V_REG_LDOSMD, U5 MAX232SOIC16, U6 ARDUINO-MEGAFULL

Commit message: got code working again
Connections:
- net MISO: now also U6.50; no longer U6.51
- net MOSI: now also U6.51; no longer U6.50
Changed lines of the file:
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@@
 <signal name="MOSI">
 <contactref element="U$1" pad="5"/>
-<contactref element="U6" pad="50"/>
-<wire x1="82.81" y1="10.795" x2="93.98" y2="12.7" width="0" layer="19" extent="1-1"/>
+<contactref element="U6" pad="51"/>
+<wire x1="82.81" y1="10.795" x2="96.52" y2="12.7" width="0" layer="19" extent="1-1"/>
 </signal>
 <signal name="SCK">
@@
 <signal name="MISO">
 <contactref element="U$5" pad="DO"/>
-<contactref element="U6" pad="51"/>
-<wire x1="88.9" y1="13.97" x2="96.52" y2="12.7" width="0" layer="19" extent="1-1"/>
+<contactref element="U6" pad="50"/>
+<wire x1="88.9" y1="13.97" x2="93.98" y2="12.7" width="0" layer="19" extent="1-1"/>
 </signal>
 <signal name="N$5">
